File: uSDX-x.sch (KiCad schematic (older format))
At the start: 89 parts, among them J1 DC Jack, J10 1602LCD, J11 Mic, J12 Headphones, J13 PA MOSFETs, J2 FilterConn, J3 Antenna, J4 Etherkit si5351, J5 EK CLK0, J6 EK CLK1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

Commit message: added first pcb layout and board photo
Parts:
- J10: footprint Connector_PinSocket_2.54mm:PinSocket_1x16_P2.54mm_Vertical -> Display:WC1602A
- J11: value Mic -> PJ-324M
- J12: value Headphones -> PJ-324M
- J3: footprint Connector_Coaxial:SMA_Amphenol_132134_Vertical -> eec:Molex-73100-0114-0-0-0
Changed lines of the file:
@@
 F 0 "J3" H 6650 3675 50  0000 L CNN
 F 1 "Antenna" H 6650 3584 50  0000 L CNN
-F 2 "Connector_Coaxial:SMA_Amphenol_132134_Vertical" H 6550 3700 50  0001 C CNN
+F 2 "eec:Molex-73100-0114-0-0-0" H 6550 3700 50  0001 C CNN
 F 3 " ~" H 6550 3700 50  0001 C CNN
 F 4 "no assembly" H 6550 3700 50  0001 C CNN "LCSC"
@@
 F 0 "J10" H 10850 6250 50  0000 L CNN
 F 1 "1602LCD" H 10750 6150 50  0000 L CNN
-F 2 "Connector_PinSocket_2.54mm:PinSocket_1x16_P2.54mm_Vertical" H 11000 5350 50  0001 C CNN
+F 2 "Display:WC1602A" H 11000 5350 50  0001 C CNN
 F 3 "~" H 11000 5350 50  0001 C CNN
 F 4 "no assembly" H 11000 5350 50  0001 C CNN "LCSC"
@@
 Text Notes 600  4650 0    50   ~ 0
 Alternate: FST3253
-$Comp
-L Connector:AudioJack3_SwitchTR J12
-U 1 1 606FED8B
-P 8900 3400
-F 0 "J12" H 8900 3600 50  0000 R CNN
-F 1 "Headphones" H 9050 3650 50  0000 R CNN
-F 2 "Connector_Audio:Jack_3.5mm_Ledino_KB3SPRS_Horizontal" H 8900 3600 50  0001 C CNN
-F 3 "~" H 8900 3600 50  0001 C CNN
-F 4 "no assembly" H 8900 3400 50  0001 C CNN "LCSC"
-	1    8900 3400
-	-1   0    0    1
-$EndComp
 Text GLabel 7800 3300 0    50   Input ~ 0
 SIDETONE
@@
 P 7750 2700
 F 0 "J11" H 7750 2900 50  0000 R CNN
-F 1 "Mic" H 7750 3000 50  0000 R CNN
+F 1 "PJ-324M" H 7850 3000 50  0000 R CNN
 F 2 "Connector_Audio:Jack_3.5mm_Ledino_KB3SPRS_Horizontal" H 7750 2900 50  0001 C CNN
-F 3 "~" H 7750 2900 50  0001 C CNN
+F 3 "https://store.comet.bg/download-file.php?id=18858" H 7750 2900 50  0001 C CNN
 F 4 "no assembly" H 7750 2700 50  0001 C CNN "LCSC"
 	1    7750 2700
@@
 U 1 1 6076E739
 P 9350 6000
-F 0 "J13" H 9378 6026 50  0000 L CNN
-F 1 "PA MOSFETs" V 9500 5700 50  0000 L CNN
+F 0 "J13" H 9250 5800 50  0000 L CNN
+F 1 "PA MOSFETs" V 9450 5700 50  0000 L CNN
 F 2 "Connector_PinSocket_2.54mm:PinSocket_1x03_P2.54mm_Vertical" H 9350 6000 50  0001 C CNN
 F 3 "~" H 9350 6000 50  0001 C CNN
@@
 	1    0    0    -1
 $EndComp
+$Comp
+L Connector:AudioJack3_SwitchTR J12
+U 1 1 606FED8B
+P 8900 3400
+F 0 "J12" H 8900 3600 50  0000 R CNN
+F 1 "PJ-324M" H 9000 3650 50  0000 R CNN
+F 2 "Connector_Audio:Jack_3.5mm_Ledino_KB3SPRS_Horizontal" H 8900 3600 50  0001 C CNN
+F 3 "~" H 8900 3600 50  0001 C CNN
+F 4 "no assembly" H 8900 3400 50  0001 C CNN "LCSC"
+	1    8900 3400
+	-1   0    0    1
+$EndComp
 $EndSCHEMATC

Commit message: files for first iteration build, some pcb layout improvements
Parts:
- J10: footprint Display:WC1602A -> uSDX-x:WC1602A
- R5: footprint Resistor_SMD:R_0805_2012Metric_Pad1.15x1.40mm_HandSolder -> Resistor_SMD:R_1206_3216Metric_Pad1.42x1.75mm_HandSolder
- SW1: footprint Button_Switch_SMD:SW_DPDT_CK_JS202011JCQN -> uSDX-x:SW_DPDT-6_3.5x9.1x2.5P
- U2: footprint Package_SO:SOIC-8_5.275x5.275mm_P1.27mm -> Package_SO:SOIC-8_3.9x4.9mm_P1.27mm
Other:
- note added: "Power: RC = 1/10 W, RE = 1/20 W\nRC 1206 SMD"
- note removed: "Power: RC = 1/10 W, RE = 1/20 W"
Changed lines of the file:
@@
 F 0 "R5" V 1445 7250 50  0000 C CNN
 F 1 "22R" V 1536 7250 50  0000 C CNN
-F 2 "Resistor_SMD:R_0805_2012Metric_Pad1.15x1.40mm_HandSolder" H 1650 7250 50  0001 C CNN
+F 2 "Resistor_SMD:R_1206_3216Metric_Pad1.42x1.75mm_HandSolder" H 1650 7250 50  0001 C CNN
 F 3 "~" H 1650 7250 50  0001 C CNN
 F 4 "C17958" H 1650 7250 50  0001 C CNN "LCSC"
@@
 F 0 "SW1" H 4000 3985 50  0000 C CNN
 F 1 "SW_DPDT_x2" H 4000 3894 50  0000 C CNN
-F 2 "Button_Switch_SMD:SW_DPDT_CK_JS202011JCQN" H 4000 3700 50  0001 C CNN
+F 2 "uSDX-x:SW_DPDT-6_3.5x9.1x2.5P" H 4000 3700 50  0001 C CNN
 F 3 "https://datasheet.lcsc.com/szlcsc/1809211421_Korean-Hroparts-Elec-K3-2245S-F1_C145844.pdf" H 4000 3700 50  0001 C CNN
 F 4 "C145844" H 4000 3700 50  0001 C CNN "LCSC"
 	1    4000 3700
 	1    0    0    -1
-$EndComp
-$Comp
-L Switch:SW_DPDT_x2 SW1
-U 2 1 613579E2
-P 6150 3700
-F 0 "SW1" H 6150 3985 50  0000 C CNN
-F 1 "SW_DPDT_x2" H 6150 3894 50  0000 C CNN
-F 2 "Button_Switch_SMD:SW_DPDT_CK_JS202011JCQN" H 6150 3700 50  0001 C CNN
-F 3 "https://datasheet.lcsc.com/szlcsc/1809211421_Korean-Hroparts-Elec-K3-2245S-F1_C145844.pdf" H 6150 3700 50  0001 C CNN
-F 4 "C145844" H 6150 3700 50  0001 C CNN "LCSC"
-	2    6150 3700
-	-1   0    0    -1
 $EndComp
 Wire Wire Line
@@
 F 0 "J10" H 10850 6250 50  0000 L CNN
 F 1 "1602LCD" H 10750 6150 50  0000 L CNN
-F 2 "Display:WC1602A" H 11000 5350 50  0001 C CNN
+F 2 "uSDX-x:WC1602A" H 11000 5350 50  0001 C CNN
 F 3 "~" H 11000 5350 50  0001 C CNN
 F 4 "no assembly" H 11000 5350 50  0001 C CNN "LCSC"
@@
 F 0 "U2" H 6500 6950 50  0000 L CNN
 F 1 "NE5532DR" H 6300 6850 50  0000 L CNN
-F 2 "Package_SO:SOIC-8_5.275x5.275mm_P1.27mm" H 6550 6850 50  0001 C CNN
+F 2 "Package_SO:SOIC-8_3.9x4.9mm_P1.27mm" H 6550 6850 50  0001 C CNN
 F 3 "http://www.ti.com/lit/ds/symlink/ne5532.pdf" H 6550 6850 50  0001 C CNN
 F 4 "C7426" H 6550 6850 50  0001 C CNN "LCSC"
@@
 F 0 "U2" H 5200 6617 50  0000 C CNN
 F 1 "NE5532DR" H 5200 6526 50  0000 C CNN
-F 2 "Package_SO:SOIC-8_5.275x5.275mm_P1.27mm" H 5200 6250 50  0001 C CNN
+F 2 "Package_SO:SOIC-8_3.9x4.9mm_P1.27mm" H 5200 6250 50  0001 C CNN
 F 3 "http://www.ti.com/lit/ds/symlink/ne5532.pdf" H 5200 6250 50  0001 C CNN
 F 4 "C7426" H 5200 6250 50  0001 C CNN "LCSC"
@@
 F 0 "U2" H 5300 5400 50  0000 C CNN
 F 1 "NE5532DR" H 5350 5700 50  0000 C CNN
-F 2 "Package_SO:SOIC-8_5.275x5.275mm_P1.27mm" H 5200 5550 50  0001 C CNN
+F 2 "Package_SO:SOIC-8_3.9x4.9mm_P1.27mm" H 5200 5550 50  0001 C CNN
 F 3 "http://www.ti.com/lit/ds/symlink/ne5532.pdf" H 5200 5550 50  0001 C CNN
 F 4 "C7426" H 5200 5550 50  0001 C CNN "LCSC"
@@
 Connection ~ 4800 3600
 Text Notes 600  7700 0    50   ~ 0
-Power: RC = 1/10 W, RE = 1/20 W
+Power: RC = 1/10 W, RE = 1/20 W\nRC 1206 SMD
 $Comp
 L power:+5V #PWR0101
@@
 	-1   0    0    1
 $EndComp
+$Comp
+L Switch:SW_DPDT_x2 SW1
+U 2 1 613579E2
+P 6150 3700
+F 0 "SW1" H 6150 3985 50  0000 C CNN
+F 1 "SW_DPDT_x2" H 6150 3894 50  0000 C CNN
+F 2 "uSDX-x:SW_DPDT-6_3.5x9.1x2.5P" H 6150 3700 50  0001 C CNN
+F 3 "https://datasheet.lcsc.com/szlcsc/1809211421_Korean-Hroparts-Elec-K3-2245S-F1_C145844.pdf" H 6150 3700 50  0001 C CNN
+F 4 "C145844" H 6150 3700 50  0001 C CNN "LCSC"
+	2    6150 3700
+	-1   0    0    -1
+$EndComp
 $EndSCHEMATC
