File: uSDX-x_asmade_042021.kicad_pcb (KiCad board)
At the start: 2 copper layers, 100 x 93.3 mm, 89 parts, among them J1 DC Jack, J10 1602LCD, J11 PJ-324M, J12 PJ-324M, J13 PA MOSFETs, J2 FilterConn, J3 Antenna, J4 Etherkit si5351, J5 EK CLK0, J6 EK CLK1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

Commit message: files for first iteration build, some pcb layout improvements
Routing:
- net +5V: track 188.6 -> 175.1 mm
- net GateDrive: track 52.0 -> 58.8 mm
- net BUTTONS: track 96.5 -> 93.3 mm, vias 0 -> 2
- net Net-(J3-Pad1): track 36.9 -> 34.9 mm
- net LCD_RS: track 208.8 -> 207.1 mm
- net LCD_D5: track 112.4 -> 111.1 mm
- net LCD_EN: track 85.9 -> 84.7 mm
- net CLK2: track 45.3 -> 46.3 mm
- net RX: track 63.6 -> 63.1 mm
