File: uSDX-x_inprog.kicad_pcb (KiCad board)
At the start: 2 copper layers, 100 x 93.3 mm, 89 parts, among them J1 DC Jack, J10 1602LCD, J11 PJ-324M, J12 PJ-324M, J13 PA MOSFETs, J2 FilterConn, J3 Antenna, J4 Etherkit si5351, J5 EK CLK0, J6 EK CLK1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

Commit message: files for first iteration build, some pcb layout improvements
Parts:
- J10: footprint uSDX-x:WC1602A -> Display:WC1602A
- R5: footprint Resistor_SMD:R_1206_3216Metric_Pad1.42x1.75mm_HandSolder -> Resistor_SMD:R_0805_2012Metric_Pad1.15x1.40mm_HandSolder
- SW1: footprint uSDX-x:SW_DPDT-6_3.5x9.1x2.5P -> Button_Switch_SMD:SW_DPDT_CK_JS202011JCQN
- U2: footprint Package_SO:SOIC-8_3.9x4.9mm_P1.27mm -> Package_SO:SOIC-8_5.275x5.275mm_P1.27mm
- moved J1 5.97 mm to (110.9, 58.6)
- moved C21 1.80 mm to (110.8, 78.4)
- moved C16 1.80 mm to (110.7, 82.4)
- moved R13 1.80 mm to (108.4, 82.4)
- moved R15 1.80 mm to (109.7, 75.2)
- moved R16 1.80 mm to (108.3, 78.4)
- moved J3 1.72 mm to (90.3, 138.3)
- moved C17 1.71 mm to (92.1, 81.0)
- moved C22 1.71 mm to (92.1, 77.0)
- moved R14 1.71 mm to (94.5, 81.0)
- moved R17 1.71 mm to (93.3, 74.0)
- moved R18 1.71 mm to (94.5, 77.0)
- moved SW1 1.18 mm to (126.1, 139.6)
- moved U2 0.62 mm to (101.4, 82.4)
- moved R5 0.56 mm to (137.1, 113.5)
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Routing:
- net CLK0: track 91.0 -> 47.5 mm
- net SIG_OUT: track 189.0 -> 153.7 mm
- net +3V3: track 191.6 -> 222.4 mm
- net CLK1: track 74.3 -> 52.2 mm, vias 2 -> 4
- net CLK2: track 45.3 -> 24.7 mm
- net Net-(C19-Pad1): track 44.0 -> 26.7 mm
- net GND: track 14.9 -> 28.7 mm
- net LCD_RS: track 208.8 -> 195.6 mm
- net +5V: track 188.6 -> 177.8 mm
- net SCL_3V3: track 175.0 -> 184.9 mm
- net RF: track 94.2 -> 89.3 mm
- net GateDrive: track 52.0 -> 48.2 mm, vias 2 -> 0
- net AUDIO2: track 33.5 -> 37.0 mm
- net BUTTONS: track 96.5 -> 93.3 mm, vias 0 -> 2
- net Net-(J3-Pad1): track 36.9 -> 33.8 mm
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- removed copper zone on F.Cu, net +12V
Other:
- board size 100 x 93.3 mm -> 100 x 89.8 mm
